Commit message: ids_camera -> camera, separate launcher for images resizing

File: monoforce_gazebo/urdf/accessories/camera.urdf.xacro (robot description, xacro)
@@ -1,6 +1,6 @@
 <?xml version="1.0"?>
 <robot xmlns:xacro="http://ros.org/wiki/xacro">
-    <xacro:macro name="ids_sensor" params="xyz rpy parent topic label">
-      <joint name="ids_joint_${label}" type="fixed">
+    <xacro:macro name="camera_sensor" params="xyz rpy parent topic label">
+      <joint name="camera_joint_${label}" type="fixed">
         <origin xyz="${xyz}" rpy="${rpy}"/>
         <parent link="${parent}"/>
@@ -11,5 +11,5 @@
       <!-- Virtual camera Z-front frame -->
       <link name="camera_${label}_gazebo"/>
-      <joint name="ids_joint_${label}_gazebo" type="fixed">
+      <joint name="camera_joint_${label}_gazebo" type="fixed">
        <parent link="camera_${label}"/>
        <child link="camera_${label}_gazebo"/>
@@ -17,5 +17,5 @@
      </joint>
       <gazebo reference="camera_${label}">
-        <sensor type="camera" name="ids_camera_${label}">
+        <sensor type="camera" name="camera_${label}">
           <update_rate>10.0</update_rate>
           <camera name="head">
@@ -39,5 +39,5 @@
             </noise>
           </camera>
-          <plugin name="ids_controller" filename="libgazebo_ros_camera.so">
+          <plugin name="camera_controller" filename="libgazebo_ros_camera.so">
             <alwaysOn>true</alwaysOn>
             <updateRate>10.0</updateRate>

File: monoforce_gazebo/urdf/husky.urdf.xacro (robot description, xacro)
@@ -26,32 +26,32 @@
   <xacro:arg name="imu_rpy"     default="$(optenv HUSKY_IMU_RPY 0 -1.5708 3.1416)"/>
   <xacro:arg name="imu_parent"  default="$(optenv HUSKY_IMU_PARENT base_link)"/>
-  <!-- FRONT IDS Camera -->
-  <xacro:arg name="ids_front_enabled"             default="$(optenv HUSKY_IDS_FRONT_ENABLED 1)" />
-  <xacro:arg name="ids_front_xyz"                 default="$(optenv HUSKY_IDS_FRONT_XYZ 0.4 0 0.1)"/>
-  <xacro:arg name="ids_front_rpy"                 default="$(optenv HUSKY_IDS_FRONT_RPY 0 0 0)"/>
-  <xacro:arg name="ids_front_parent"              default="$(optenv HUSKY_IDS_FRONT_PARENT top_plate_link)"/>
-  <xacro:arg name="ids_front_topic"               default="$(optenv HUSKY_IDS_FRONT_TOPIC ids_camera)"/>
-  <xacro:arg name="ids_front_label"               default="$(optenv HUSKY_IDS_FRONT_LABEL front)"/>
-  <!-- Left IDS Camera -->
-  <xacro:arg name="ids_left_enabled"               default="$(optenv HUSKY_IDS_LEFT_ENABLED 1)" />
-  <xacro:arg name="ids_left_xyz"                   default="$(optenv HUSKY_IDS_LEFT_XYZ 0 0.2 0.1)"/>
-  <xacro:arg name="ids_left_rpy"                   default="$(optenv HUSKY_IDS_LEFT_RPY 0 0 1.57)"/>
-  <xacro:arg name="ids_left_parent"                default="$(optenv HUSKY_IDS_LEFT_PARENT top_plate_link)"/>
-  <xacro:arg name="ids_left_topic"                 default="$(optenv HUSKY_IDS_LEFT_TOPIC ids_camera)"/>
-  <xacro:arg name="ids_left_label"                 default="$(optenv HUSKY_IDS_LEFT_LABEL left)"/>
-  <!-- Right IDS Camera -->
-  <xacro:arg name="ids_right_enabled"              default="$(optenv HUSKY_IDS_RIGHT_ENABLED 1)" />
-  <xacro:arg name="ids_right_xyz"                  default="$(optenv HUSKY_IDS_RIGHT_XYZ 0 -0.2 0.1)"/>
-  <xacro:arg name="ids_right_rpy"                  default="$(optenv HUSKY_IDS_RIGHT_RPY 0 0 -1.57)"/>
-  <xacro:arg name="ids_right_parent"               default="$(optenv HUSKY_IDS_RIGHT_PARENT top_plate_link)"/>
-  <xacro:arg name="ids_right_topic"                default="$(optenv HUSKY_IDS_RIGHT_TOPIC ids_camera)"/>
-  <xacro:arg name="ids_right_label"                default="$(optenv HUSKY_IDS_RIGHT_LABEL right)"/>
-  <!-- Rear IDS Camera -->
-  <xacro:arg name="ids_rear_enabled"               default="$(optenv HUSKY_IDS_REAR_ENABLED 1)" />
-  <xacro:arg name="ids_rear_xyz"                   default="$(optenv HUSKY_IDS_REAR_XYZ -0.4 0 0.1)"/>
-  <xacro:arg name="ids_rear_rpy"                   default="$(optenv HUSKY_IDS_REAR_RPY 0 0 3.14)"/>
-  <xacro:arg name="ids_rear_parent"                default="$(optenv HUSKY_IDS_REAR_PARENT top_plate_link)"/>
-  <xacro:arg name="ids_rear_topic"                 default="$(optenv HUSKY_IDS_REAR_TOPIC ids_camera)"/>
-  <xacro:arg name="ids_rear_label"                 default="$(optenv HUSKY_IDS_REAR_LABEL rear)"/>
+  <!-- FRONT Camera -->
+  <xacro:arg name="camera_front_enabled"             default="$(optenv HUSKY_camera_FRONT_ENABLED 1)" />
+  <xacro:arg name="camera_front_xyz"                 default="$(optenv HUSKY_camera_FRONT_XYZ 0.4 0 0.1)"/>
+  <xacro:arg name="camera_front_rpy"                 default="$(optenv HUSKY_camera_FRONT_RPY 0 0 0)"/>
+  <xacro:arg name="camera_front_parent"              default="$(optenv HUSKY_camera_FRONT_PARENT top_plate_link)"/>
+  <xacro:arg name="camera_front_topic"               default="$(optenv HUSKY_camera_FRONT_TOPIC camera)"/>
+  <xacro:arg name="camera_front_label"               default="$(optenv HUSKY_camera_FRONT_LABEL front)"/>
+  <!-- Left Camera -->
+  <xacro:arg name="camera_left_enabled"               default="$(optenv HUSKY_camera_LEFT_ENABLED 1)" />
+  <xacro:arg name="camera_left_xyz"                   default="$(optenv HUSKY_camera_LEFT_XYZ 0 0.2 0.1)"/>
+  <xacro:arg name="camera_left_rpy"                   default="$(optenv HUSKY_camera_LEFT_RPY 0 0 1.57)"/>
+  <xacro:arg name="camera_left_parent"                default="$(optenv HUSKY_camera_LEFT_PARENT top_plate_link)"/>
+  <xacro:arg name="camera_left_topic"                 default="$(optenv HUSKY_camera_LEFT_TOPIC camera)"/>
+  <xacro:arg name="camera_left_label"                 default="$(optenv HUSKY_camera_LEFT_LABEL left)"/>
+  <!-- Right Camera -->
+  <xacro:arg name="camera_right_enabled"              default="$(optenv HUSKY_camera_RIGHT_ENABLED 1)" />
+  <xacro:arg name="camera_right_xyz"                  default="$(optenv HUSKY_camera_RIGHT_XYZ 0 -0.2 0.1)"/>
+  <xacro:arg name="camera_right_rpy"                  default="$(optenv HUSKY_camera_RIGHT_RPY 0 0 -1.57)"/>
+  <xacro:arg name="camera_right_parent"               default="$(optenv HUSKY_camera_RIGHT_PARENT top_plate_link)"/>
+  <xacro:arg name="camera_right_topic"                default="$(optenv HUSKY_camera_RIGHT_TOPIC camera)"/>
+  <xacro:arg name="camera_right_label"                default="$(optenv HUSKY_camera_RIGHT_LABEL right)"/>
+  <!-- Rear Camera -->
+  <xacro:arg name="camera_rear_enabled"               default="$(optenv HUSKY_camera_REAR_ENABLED 1)" />
+  <xacro:arg name="camera_rear_xyz"                   default="$(optenv HUSKY_camera_REAR_XYZ -0.4 0 0.1)"/>
+  <xacro:arg name="camera_rear_rpy"                   default="$(optenv HUSKY_camera_REAR_RPY 0 0 3.14)"/>
+  <xacro:arg name="camera_rear_parent"                default="$(optenv HUSKY_camera_REAR_PARENT top_plate_link)"/>
+  <xacro:arg name="camera_rear_topic"                 default="$(optenv HUSKY_camera_REAR_TOPIC camera)"/>
+  <xacro:arg name="camera_rear_label"                 default="$(optenv HUSKY_camera_REAR_LABEL rear)"/>
   <!-- LiDAR -->
   <xacro:arg name="ouster_enabled"              default="$(optenv HUSKY_OUSTER_ENABLED 1)" />
@@ -72,5 +72,5 @@
   <xacro:property name="gpu" value="$(arg gpu)" />
   <!-- Included URDF/XACRO Files -->
-  <xacro:include filename="$(find monoforce_gazebo)/urdf/accessories/ids_camera.urdf.xacro"/>
+  <xacro:include filename="$(find monoforce_gazebo)/urdf/accessories/camera.urdf.xacro"/>
   <xacro:include filename="$(find monoforce_gazebo)/urdf/accessories/ouster_lidar.urdf.xacro"/>
   <xacro:include filename="$(find ouster_description)/urdf/OS0-32.urdf.xacro"/>
@@ -146,36 +146,36 @@
   <!-- Husky Decorations -->
   <xacro:husky_decorate />
-  <!-- IDS Cameras -->
-  <xacro:if value="$(arg ids_front_enabled)">
-      <xacro:ids_sensor xyz="$(arg ids_front_xyz)"
-                        rpy="$(arg ids_front_rpy)"
-                        parent="$(arg ids_front_parent)"
-                        topic="$(arg ids_front_topic)"
-                        label="$(arg ids_front_label)">
-      </xacro:ids_sensor>
-  </xacro:if>
-  <xacro:if value="$(arg ids_left_enabled)">
-      <xacro:ids_sensor xyz="$(arg ids_left_xyz)"
-                          rpy="$(arg ids_left_rpy)"
-                          parent="$(arg ids_left_parent)"
-                          topic="$(arg ids_left_topic)"
-                          label="$(arg ids_left_label)">
-      </xacro:ids_sensor>
-  </xacro:if>
-  <xacro:if value="$(arg ids_right_enabled)">
-      <xacro:ids_sensor xyz="$(arg ids_right_xyz)"
-                          rpy="$(arg ids_right_rpy)"
-                          parent="$(arg ids_right_parent)"
-                          topic="$(arg ids_right_topic)"
-                          label="$(arg ids_right_label)">
-      </xacro:ids_sensor>
-  </xacro:if>
-  <xacro:if value="$(arg ids_rear_enabled)">
-      <xacro:ids_sensor xyz="$(arg ids_rear_xyz)"
-                          rpy="$(arg ids_rear_rpy)"
-                          parent="$(arg ids_rear_parent)"
-                          topic="$(arg ids_rear_topic)"
-                          label="$(arg ids_rear_label)">
-      </xacro:ids_sensor>
+  <!-- Cameras -->
+  <xacro:if value="$(arg camera_front_enabled)">
+      <xacro:camera_sensor xyz="$(arg camera_front_xyz)"
+                        rpy="$(arg camera_front_rpy)"
+                        parent="$(arg camera_front_parent)"
+                        topic="$(arg camera_front_topic)"
+                        label="$(arg camera_front_label)">
+      </xacro:camera_sensor>
+  </xacro:if>
+  <xacro:if value="$(arg camera_left_enabled)">
+      <xacro:camera_sensor xyz="$(arg camera_left_xyz)"
+                          rpy="$(arg camera_left_rpy)"
+                          parent="$(arg camera_left_parent)"
+                          topic="$(arg camera_left_topic)"
+                          label="$(arg camera_left_label)">
+      </xacro:camera_sensor>
+  </xacro:if>
+  <xacro:if value="$(arg camera_right_enabled)">
+      <xacro:camera_sensor xyz="$(arg camera_right_xyz)"
+                          rpy="$(arg camera_right_rpy)"
+                          parent="$(arg camera_right_parent)"
+                          topic="$(arg camera_right_topic)"
+                          label="$(arg camera_right_label)">
+      </xacro:camera_sensor>
+  </xacro:if>
+  <xacro:if value="$(arg camera_rear_enabled)">
+      <xacro:camera_sensor xyz="$(arg camera_rear_xyz)"
+                          rpy="$(arg camera_rear_rpy)"
+                          parent="$(arg camera_rear_parent)"
+                          topic="$(arg camera_rear_topic)"
+                          label="$(arg camera_rear_label)">
+      </xacro:camera_sensor>
   </xacro:if>
   <!-- Ouster LiDAR -->
